File: kicad/handwire microboard.kicad_pcb (KiCad board)
At the start: 2 copper layers, 34.1 x 47.3 mm, 11 parts, among them J1 ProMicro18pin, J2 ProMicro18pin, J3 EliteC5pin, SW1 SW_Push, T1 AudioJack4, T2 AudioJack4, U1 Elite-C

Commit message: fixed issue and update files
Parts:
- removed H3, H4: MountingHole, MountingHole:MountingHole_2.2mm_M2
- removed J3: EliteC5pin, Connector_PinHeader_2.54mm:PinHeader_1x07_P2.54mm_Vertical
- added T3: AudioJack4, DreaM117er-keebLibrary:TRRS-PJ-320A, F.Cu at (21.9, 20.4)
- added T4: AudioJack4, DreaM117er-keebLibrary:TRRS-PJ-320A, F.Cu at (49.5, 61.3)
- J1: footprint Connector_PinHeader_2.54mm:PinHeader_2x09_P2.54mm_Vertical -> DreaM117er-keebLibrary:PinHeader_2x09_P2.54mm_Vertical_Rside; moved to B.Cu
- J2: footprint Connector_PinHeader_2.54mm:PinHeader_2x09_P2.54mm_Vertical -> DreaM117er-keebLibrary:PinHeader_2x09_P2.54mm_Vertical_Rside
- SW1: footprint Button_Switch_THT:SW_PUSH_6mm_H4.3mm -> Marby_kbd_footprint-main:ResetSW_1side
- T1, T2: footprint Keebio-Parts:TRRS-PJ-320A, dual side (fix) -> DreaM117er-keebLibrary:TRRS-PJ-320A
- U1: value Elite-C -> ProMicro; footprint DreaM117er-keebLibrary:Elite-C -> DreaM117er-keebLibrary:ProMicro
- moved SW1 3.48 mm to (34.9, 55.8)
- moved J1 2.54 mm to (22.3, 34.7), turned to 180 degrees
Connections:
- T1 pad 1: VCC -> unconnected-(T1-SLEEVE-Pad1)
- T1 pad 2: VCC -> D2
- T1 pad 4: D2 -> VCC
- T2 pad 1: VCC -> unconnected-(T2-SLEEVE-Pad1)
- T2 pad 2: VCC -> D2
- T2 pad 4: D2 -> VCC
Routing:
- net RESET: track 65.8 -> 50.4 mm, vias 3 -> 2
- net D2: track 88.5 -> 103.7 mm
- net VCC: track 64.5 -> 71.2 mm
- net GND: track 80.1 -> 83.6 mm
- net F1: track 3.36 -> 0.00 mm
- net F0: track 3.36 -> 0.00 mm
- net D5: track 3.36 -> 0.00 mm
- net C7: track 3.36 -> 0.00 mm
- net B7: track 3.36 -> 0.00 mm
- net D3: track 39.3 -> 40.0 mm, vias 0 -> 1

Commit message: update files
Routing:
- net GND: track 83.6 -> 0.06 mm
Changed lines of the file:
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@@
   (segment (start 41.255 41.02) (end 42.505 39.77) (width 0.25) (layer "F.Cu") (net 17))
   (segment (start 26.856105 41.02) (end 41.255 41.02) (width 0.25) (layer "F.Cu") (net 17))
-  (segment (start 42.505 27.07) (end 46.98 27.07) (width 0.35) (layer "F.Cu") (net 18))
-  (segment (start 42.505 27.07) (end 29.805 27.07) (width 0.35) (layer "F.Cu") (net 18))
-  (segment (start 47.4865 26.5635) (end 50.235 26.5635) (width 0.35) (layer "F.Cu") (net 18))
-  (segment (start 29.805 27.07) (end 27.265 29.61) (width 0.35) (layer "F.Cu") (net 18))
-  (segment (start 46.98 27.07) (end 47.4865 26.5635) (width 0.35) (layer "F.Cu") (net 18))
-  (segment (start 40.96 55.84) (end 43.335 58.215) (width 0.35) (layer "B.Cu") (net 18))
-  (segment (start 36.505 57.47) (end 38.135 55.84) (width 0.35) (layer "B.Cu") (net 18))
   (segment (start 27.265 29.61) (end 27.2015 29.61) (width 0.35) (layer "B.Cu") (net 18))
-  (segment (start 25.49 54.06) (end 25.49 33.925) (width 0.35) (layer "B.Cu") (net 18))
-  (segment (start 26.455 58.97) (end 27.955 57.47) (width 0.35) (layer "B.Cu") (net 18))
-  (segment (start 43.335 58.215) (end 43.335 63.57) (width 0.35) (layer "B.Cu") (net 18))
-  (segment (start 26.455 58.97) (end 26.455 55.025) (width 0.35) (layer "B.Cu") (net 18))
-  (segment (start 25.49 33.925) (end 27.265 32.15) (width 0.35) (layer "B.Cu") (net 18))
-  (segment (start 26.455 55.025) (end 25.49 54.06) (width 0.35) (layer "B.Cu") (net 18))
-  (segment (start 38.135 55.84) (end 40.96 55.84) (width 0.35) (layer "B.Cu") (net 18))
-  (segment (start 27.2015 29.61) (end 24.155 26.5635) (width 0.35) (layer "B.Cu") (net 18))
-  (segment (start 27.955 57.47) (end 36.505 57.47) (width 0.35) (layer "B.Cu") (net 18))
-  (segment (start 27.265 29.61) (end 27.265 32.15) (width 0.35) (layer "B.Cu") (net 18))
   (segment (start 23.941 34.06) (end 24.74 34.06) (width 0.25) (layer "F.Cu") (net 19))
   (segment (start 26.34 30.88) (end 41.235 30.88) (width 0.25) (layer "F.Cu") (net 19))
@@
         (xy 52.74 66.04)
         (xy 17.18 66.04)
-        (xy 17.18 66.04)
       )
     )
@@
   )
   (zone (net 0) (net_name "") (layer "B.Cu") (name "GND") (hatch edge 0.5)
+    (priority 2)
+    (connect_pads (clearance 0.5))
+    (min_thickness 0.25) (filled_areas_thickness no)
+    (fill (thermal_gap 0.5) (thermal_bridge_width 0.5) (island_removal_mode 1) (island_area_min 10))
+    (polygon
+      (pts
+        (xy 22.88 30.98)
+        (xy 24.57 32.89)
+        (xy 22.96 34.1)
+        (xy 22.45 33.86)
+      )
+    )
+  )
+  (zone (net 0) (net_name "") (layer "B.Cu") (name "GND") (hatch edge 0.5)
     (priority 4)
     (connect_pads (clearance 0.5))
@@
       )
     )
-  )
-  (zone (net 0) (net_name "") (layer "B.Cu") (name "GND") (hatch edge 0.5)
-    (priority 2)
-    (connect_pads (clearance 0.5))
-    (min_thickness 0.25) (filled_areas_thickness no)
-    (fill (thermal_gap 0.5) (thermal_bridge_width 0.5) (island_removal_mode 1) (island_area_min 10))
-    (polygon
-      (pts
-        (xy 22.57 30.01)
-        (xy 25.77 25.16)
-        (xy 27.31 31.49)
-        (xy 24.6 33.84)
-        (xy 22.63 33.71)
-      )
-    )

Commit message: update files
Parts:
- SW1: footprint Marby_kbd_footprint-main:ResetSW_1side -> DreaM117er-keebLibrary:ResetSW_1side
Routing:
- net GND: track 0.06 -> 83.8 mm
- added copper zone on F.Cu, net GND
Changed lines of the file:
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@@
     )
   )
-  (footprint "Marby_kbd_footprint-main:ResetSW_1side" (layer "F.Cu")
+  (footprint "DreaM117er-keebLibrary:ResetSW_1side" (layer "F.Cu")
     (at 34.885 55.84)
     (property "Sheetfile" "handwire microboard.kicad_sch")
@@
         (effects (font (size 1.27 1.524) (thickness 0.2032)))
     )
+    (fp_text user "GND" (at -6.35 5.461) (layer "B.SilkS")
+        (effects (font (size 0.8 0.8) (thickness 0.15)) (justify mirror))
+    )
+    (fp_text user "GND" (at -11.43 -5.461) (layer "B.SilkS")
+        (effects (font (size 0.8 0.8) (thickness 0.15)) (justify mirror))
+    )
     (fp_text user "VCC" (at -6.35 -5.461) (layer "B.SilkS")
         (effects (font (size 0.8 0.8) (thickness 0.15)) (justify mirror))
     )
-    (fp_text user "GND" (at -6.35 5.461) (layer "B.SilkS")
-        (effects (font (size 0.8 0.8) (thickness 0.15)) (justify mirror))
-    )
     (fp_text user "RST" (at -8.91 -5.48) (layer "B.SilkS")
         (effects (font (size 0.8 0.8) (thickness 0.15)) (justify mirror))
@@
         (effects (font (size 0.8 0.8) (thickness 0.15)) (justify mirror))
     )
-    (fp_text user "GND" (at -11.43 -5.461) (layer "B.SilkS")
-        (effects (font (size 0.8 0.8) (thickness 0.15)) (justify mirror))
+    (fp_text user "GND" (at -8.89 5.461) (layer "F.SilkS")
+        (effects (font (size 0.8 0.8) (thickness 0.15)))
+    )
+    (fp_text user "GND" (at -6.35 5.461) (layer "F.SilkS")
+        (effects (font (size 0.8 0.8) (thickness 0.15)))
+    )
+    (fp_text user "VCC" (at -6.35 -5.461) (layer "F.SilkS")
+        (effects (font (size 0.8 0.8) (thickness 0.15)))
+    )
+    (fp_text user "RST" (at -8.92 -5.34) (layer "F.SilkS")
+        (effects (font (size 0.8 0.8) (thickness 0.15)))
     )
     (fp_text user "GND" (at -11.43 -5.461) (layer "F.SilkS")
-        (effects (font (size 0.8 0.8) (thickness 0.15)))
-    )
-    (fp_text user "RST" (at -8.92 -5.34) (layer "F.SilkS")
-        (effects (font (size 0.8 0.8) (thickness 0.15)))
-    )
-    (fp_text user "VCC" (at -6.35 -5.461) (layer "F.SilkS")
-        (effects (font (size 0.8 0.8) (thickness 0.15)))
-    )
-    (fp_text user "GND" (at -6.35 5.461) (layer "F.SilkS")
-        (effects (font (size 0.8 0.8) (thickness 0.15)))
-    )
-    (fp_text user "GND" (at -8.89 5.461) (layer "F.SilkS")
         (effects (font (size 0.8 0.8) (thickness 0.15)))
     )
@@
   (segment (start 41.255 41.02) (end 42.505 39.77) (width 0.25) (layer "F.Cu") (net 17))
   (segment (start 26.856105 41.02) (end 41.255 41.02) (width 0.25) (layer "F.Cu") (net 17))
-  (segment (start 27.265 29.61) (end 27.2015 29.61) (width 0.35) (layer "B.Cu") (net 18))
+  (segment (start 43.0115 26.5635) (end 50.235 26.5635) (width 0.35) (layer "F.Cu") (net 18))
+  (segment (start 27.265 29.61) (end 39.965 29.61) (width 0.35) (layer "F.Cu") (net 18))
+  (segment (start 42.505 27.07) (end 43.0115 26.5635) (width 0.35) (layer "F.Cu") (net 18))
+  (segment (start 39.965 29.61) (end 42.505 27.07) (width 0.35) (layer "F.Cu") (net 18))
+  (segment (start 26.455 58.97) (end 27.975 57.45) (width 0.35) (layer "B.Cu") (net 18))
+  (segment (start 27.265 32.15) (end 25.4905 33.9245) (width 0.35) (layer "B.Cu") (net 18))
+  (segment (start 25.4905 33.9245) (end 25.4905 54.662682) (width 0.35) (layer "B.Cu") (net 18))
+  (segment (start 41.33 55.84) (end 43.335 57.845) (width 0.35) (layer "B.Cu") (net 18))
+  (segment (start 27.265 29.61) (end 24.2185 26.5635) (width 0.35) (layer "B.Cu") (net 18))
+  (segment (start 27.975 57.45) (end 36.525 57.45) (width 0.35) (layer "B.Cu") (net 18))
+  (segment (start 26.455 55.627182) (end 26.455 58.97) (width 0.35) (layer "B.Cu") (net 18))
+  (segment (start 25.4905 54.662682) (end 26.455 55.627182) (width 0.35) (layer "B.Cu") (net 18))
+  (segment (start 38.135 55.84) (end 41.33 55.84) (width 0.35) (layer "B.Cu") (net 18))
+  (segment (start 43.335 57.845) (end 43.335 63.57) (width 0.35) (layer "B.Cu") (net 18))
+  (segment (start 27.265 29.61) (end 27.265 32.15) (width 0.35) (layer "B.Cu") (net 18))
+  (segment (start 36.525 57.45) (end 38.135 55.84) (width 0.35) (layer "B.Cu") (net 18))
+  (segment (start 24.2185 26.5635) (end 24.155 26.5635) (width 0.35) (layer "B.Cu") (net 18))
   (segment (start 23.941 34.06) (end 24.74 34.06) (width 0.25) (layer "F.Cu") (net 19))
   (segment (start 26.34 30.88) (end 41.235 30.88) (width 0.25) (layer "F.Cu") (net 19))
@@
     )
   )
+  (zone (net 18) (net_name "GND") (layer "F.Cu") (name "GND") (hatch edge 0.5)
+    (priority 9)
+    (connect_pads (clearance 0.5))
+    (min_thickness 0.25) (filled_areas_thickness no)
+    (fill (thermal_gap 0.5) (thermal_bridge_width 0.5) (island_removal_mode 1) (island_area_min 10))
+    (polygon
+      (pts
+        (xy 40.13 29.81)
+        (xy 41.29 29.1)
+        (xy 41.72 30.04)
+        (xy 40.2 30.84)
+      )
+    )
+  )
   (zone (net 0) (net_name "") (layer "F.Cu") (name "GND") (hatch edge 0.5)
     (priority 8)
@@
     )
   )
-  (zone (net 0) (net_name "") (layer "F.Cu") (name "GND") (hatch edge 0.5)
-    (priority 9)
-    (connect_pads (clearance 0.5))
-    (min_thickness 0.25) (filled_areas_thickness no)
-    (fill (thermal_gap 0.5) (thermal_bridge_width 0.5) (island_removal_mode 1) (island_area_min 10))
-    (polygon
-      (pts
-        (xy 27.97 33.78)
-        (xy 38.31 32.72)
-        (xy 41.82 34.23)
-        (xy 41.99 51.38)
-        (xy 27.83 51.2)
-      )
-    )
-  )
   (zone (net 0) (net_name "") (layers "F&B.Cu") (name "GND") (hatch edge 0.5)
     (connect_pads (clearance 0.5))
@@
         (xy 52.74 66.04)
         (xy 17.18 66.04)
-      )
-    )
-  )
-  (zone (net 0) (net_name "") (layer "B.Cu") (name "GND") (hatch edge 0.5)
-    (priority 10)
-    (connect_pads (clearance 0.5))
-    (min_thickness 0.25) (filled_areas_thickness no)
-    (fill (thermal_gap 0.5) (thermal_bridge_width 0.5) (island_removal_mode 1) (island_area_min 10))
-    (polygon
-      (pts
-        (xy 27.49 33.54)
-        (xy 42.26 34.02)
-        (xy 42.37 50.89)
-        (xy 27.42 51.17)
       )
     )
@@
   )
   (zone (net 0) (net_name "") (layer "B.Cu") (name "GND") (hatch edge 0.5)
+    (priority 11)
+    (connect_pads (clearance 0.5))
+    (min_thickness 0.25) (filled_areas_thickness no)
+    (fill (thermal_gap 0.5) (thermal_bridge_width 0.5) (island_removal_mode 1) (island_area_min 10))
+    (polygon
+      (pts
+        (xy 24.77 29.61)
+        (xy 26 29)
+        (xy 26.75 31.11)
+        (xy 25.44 33.56)
+        (xy 24.57 32.89)
+      )
+    )
+  )
+  (zone (net 0) (net_name "") (layer "B.Cu") (name "GND") (hatch edge 0.5)
     (priority 3)
     (connect_pads (clearance 0.5))
@@
       )
     )
+  )
+  (zone (net 0) (net_name "") (layer "B.Cu") (name "GND") (hatch edge 0.5)
+    (priority 10)
+    (connect_pads (clearance 0.5))
+    (min_thickness 0.25) (filled_areas_thickness no)
+    (fill (thermal_gap 0.5) (thermal_bridge_width 0.5) (island_removal_mode 1) (island_area_min 10))
+    (polygon
+      (pts
+        (xy 21.68 55.84)
+        (xy 23.56 55.34)
+        (xy 26.36 57.95)
+        (xy 24.18 59.01)
+        (xy 21.29 56.24)
+      )
+    )

Commit message: update new design file
Parts:
- moved SW1 4.50 mm to (34.9, 60.3), turned to -90 degrees
Connections:
- T1 pad 1: unconnected-(T1-SLEEVE-Pad1) -> VCC
- T1 pad 4: VCC -> unconnected-(T1-S/No-Pad4)
- T2 pad 1: unconnected-(T2-SLEEVE-Pad1) -> VCC
- T2 pad 4: VCC -> unconnected-(T2-S/No-Pad4)
- T3 pad 1: unconnected-(T3-SLEEVE-Pad1) -> VCC
- T3 pad 4: VCC -> unconnected-(T3-S/No-Pad4)
- T4 pad 1: unconnected-(T4-SLEEVE-Pad1) -> VCC
- T4 pad 4: VCC -> unconnected-(T4-S/No-Pad4)
Routing:
- net GND: track 83.8 -> 0.00 mm
- net D2: track 103.7 -> 107.5 mm, vias 1 -> 2
- net D3: track 40.0 -> 43.6 mm
- net RESET: track 50.4 -> 53.9 mm
- added copper zone on B.Cu, net GND
- removed copper zone on B.Cu, net (none)
- removed copper zone on F.Cu, net (none)

Commit message: new design
Parts:
- added ON: Jumper_Fside, DreaM117er-keebLibrary:SolderJumper-3_P1.3mm_Open_Pad0.7.x1.0mm_NumberLabels, F.Cu at (38.3, 32.1)
- added ON: Jumper_Bside, DreaM117er-keebLibrary:SolderJumper-3_P1.3mm_Open_Pad0.7.x1.0mm_NumberLabels, B.Cu at (31.5, 32.1)
- T1, T2, T3, T4: footprint DreaM117er-keebLibrary:TRRS-PJ-320A -> DreaM117er-keebLibrary:TRRS-PJ-320A, dual side
Connections:
- T1 pad 1: VCC -> A
- T1 pad 4: unconnected-(T1-S/No-Pad4) -> B
- T2 pad 1: VCC -> A
- T2 pad 4: unconnected-(T2-S/No-Pad4) -> B
- T3 pad 1: VCC -> A
- T3 pad 4: unconnected-(T3-S/No-Pad4) -> B
- T4 pad 1: VCC -> A
- T4 pad 4: unconnected-(T4-S/No-Pad4) -> B
Routing:
- net A: track 0.00 -> 78.1 mm, vias 0 -> 2
- net B: track 0.00 -> 72.6 mm, vias 0 -> 2
- net D2: track 107.5 -> 164.7 mm, vias 2 -> 3
- net VCC: track 71.0 -> 15.2 mm, vias 2 -> 0
- net F4: track 27.2 -> 55.3 mm
- net D1: track 33.4 -> 60.4 mm
- net F5: track 27.2 -> 51.2 mm
- net D0: track 33.4 -> 56.3 mm
- net F6: track 27.2 -> 47.2 mm
- net D4: track 33.4 -> 52.2 mm
- net RESET: track 53.9 -> 35.9 mm, vias 2 -> 1
- net C6: track 33.4 -> 49.8 mm
- net F7: track 27.2 -> 43.1 mm
- net D7: track 33.4 -> 45.7 mm
- net B1: track 27.2 -> 39.0 mm
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