File: kicad/handwire microboard.kicad_sch (KiCad schematic)
At the start: 9 parts, among them J1 ProMicro18pin, J2 ProMicro18pin, J3 EliteC5pin, SW1 SW_Push, T1 AudioJack4, T2 AudioJack4, U1 Elite-C

Commit message: fixed issue and update files
Parts:
- removed H3, H4: MountingHole, MountingHole:MountingHole_2.2mm_M2, symbol Mechanical:MountingHole
- removed J3: EliteC5pin, DreaM117er-keebLibrary:PinHeader_1x07_P2.54mm_Vertical_HWMB, symbol Connector:Conn_01x07_Pin
- added T3, T4: AudioJack4, DreaM117er-keebLibrary:TRRS-PJ-320A, symbol keebio:TRRS
- J1, J2: footprint DreaM117er-keebLibrary:PinHeader_2x09_P2.54mm_Vertical_HWMB -> DreaM117er-keebLibrary:PinHeader_2x09_P2.54mm_Vertical_Rside
- SW1: footprint Button_Switch_THT:SW_PUSH_6mm_H4.3mm -> DreaM117er-keebLibrary:ResetSW_1side
- T1, T2: footprint DreaM117er-keebLibrary:TRRS-PJ-320A, dual side (fix) -> DreaM117er-keebLibrary:TRRS-PJ-320A
- U1: value Elite-C -> ProMicro
Connections:
- net D2: now also T1.2 (TIP), T2.2 (TIP), T3.2 (TIP), T4.2 (TIP); no longer T1.4 (RING2), T2.4 (RING2)
- net GND: now also T3.3 (RING1), T4.3 (RING1)
- net VCC: now also T1.4 (RING2), T2.4 (RING2), T3.4 (RING2), T4.4 (RING2); no longer T1.1 (SLEEVE), T1.2 (TIP), T2.1 (SLEEVE), T2.2 (TIP)
- removed net B7: U1.25 (12/B7)
- removed net C7: U1.27 (14/C7)
- removed net D5: U1.26 (13/D5)
- removed net F0: U1.29 (16/F0)
- removed net F1: U1.28 (15/F1)
- no-connect marks 0 -> 4

Commit message: update files
Parts:
- U1: footprint DreaM117er-keebLibrary:Elite-C -> DreaM117er-keebLibrary:ProMicro
Changed lines of the file:
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@@
       (effects (font (size 1.524 1.524)))
     )
-    (property "Footprint" "DreaM117er-keebLibrary:Elite-C" (at 116.205 78.105 90)
+    (property "Footprint" "DreaM117er-keebLibrary:ProMicro" (at 116.205 78.105 90)
       (effects (font (size 1.524 1.524)) hide)
     )

Commit message: update new design file
Parts:
- T1, T2, T3, T4: symbol keebio:TRRS -> DreaM117er_Library:TRRS
Connections:
- net VCC: now also T1.1 (T/VCC), T2.1 (T/VCC), T3.1 (T/VCC), T4.1 (T/VCC); no longer T1.4 (RING2), T2.4 (RING2), T3.4 (RING2), T4.4 (RING2)

Commit message: new design
Parts:
- added JP1: Jumper_Fside, DreaM117er-keebLibrary:SolderJumper-3_P1.3mm_Open_Pad0.7.x1.0mm_NumberLabels, symbol Jumper:Jumper_3_Open
- added JP2: Jumper_Bside, DreaM117er-keebLibrary:SolderJumper-3_P1.3mm_Open_Pad0.7.x1.0mm_NumberLabels, symbol Jumper:Jumper_3_Open
- T1, T2, T3, T4: footprint DreaM117er-keebLibrary:TRRS-PJ-320A -> DreaM117er-keebLibrary:TRRS-PJ-320A, dual side
Connections:
- net VCC: now also JP1.2 (C), JP2.2 (C); no longer T1.1 (T/VCC), T2.1 (T/VCC), T3.1 (T/VCC), T4.1 (T/VCC)
- net B: now reaches T1.4 (S/No)
- net B: now also T2.4 (S/No), T3.4 (S/No), T4.4 (S/No), JP1.3 (B), JP2.3 (B)
- new net A: JP1.1 (A), JP2.1 (A), T1.1 (T/VCC), T2.1 (T/VCC), T3.1 (T/VCC), T4.1 (T/VCC)
- no-connect marks 4 -> 0
Other:
- moved on the sheet: J1, J2, SW1, T1, T2, T3, T4, U1
